Commit message: V0.0.2 - Created mimic constraint between first two joints of each finger, and renamed the joints to _Flexor to reflect actual mechanics.

File: urdf/dexhandv2_cobot_right.urdf (robot description, URDF)
Before this commit: robot dexhandv2_cobot_right, 25 links, 24 joints
Joints:
- removed joint Index_DIP
- removed joint Index_PIP
- removed joint Index_Pitch
- removed joint Index_Yaw
- removed joint Middle_DIP
- removed joint Middle_PIP
- removed joint Middle_Pitch
- removed joint Middle_Yaw
- removed joint Pinky_DIP
- removed joint Pinky_PIP
- removed joint Pinky_Pitch
- removed joint Pinky_Yaw
- removed joint Rigid 28
- removed joint Rigid 30
- removed joint Rigid 31
- removed joint Ring_DIP
- removed joint Ring_PIP
- removed joint Ring_Pitch
- removed joint Ring_Yaw
- removed joint Thumb_DIP
- removed joint Thumb_PIP
- removed joint Thumb_Pitch
- removed joint Thumb_Roll
- removed joint Thumb_Yaw
- added joint R_Index_DIP: type revolute, parent Index_Middle_1, child Index_Tip_1, origin xyz=-0.000221 -0.004184 0.030002 rpy=0 0 0, axis 0.087537 0.996161 -0.000428, limit lower=0.0 upper=1.047198 effort=100 velocity=100, mimic joint=R_Index_Flexor multiplier=1 offset=0
- added joint R_Index_Flexor: type revolute, parent Index_Knuckle_1, child Index_Middle_1, origin xyz=-0.003532 0.002993 0.045018 rpy=0 0 0, axis 0.087537 0.996161 -0.000428, limit lower=0.0 upper=1.047198 effort=100 velocity=100
- added joint R_Index_Pitch: type revolute, parent Index_Knuckle_Cross_1, child Index_Knuckle_1, origin xyz=-0.007032 0.005438 0.004034 rpy=0 0 0, axis 0.087537 0.996161 -0.000428, limit lower=0.0 upper=1.308997 effort=100 velocity=100
- added joint R_Index_Yaw: type revolute, parent Palm_1, child Index_Knuckle_Cross_1, origin xyz=0.01778 0.050623 0.084894 rpy=0 0 0, axis 0.996149 -0.087538 -0.004875, limit lower=-0.349066 upper=0.349066 effort=100 velocity=100
- added joint R_Middle_DIP: type revolute, parent Middle_Middle_1, child Midle_Tip_1, origin xyz=0.0 -0.0042 0.03 rpy=0 0 0, axis -0.0 1.0 -0.0, limit lower=0.0 upper=1.047198 effort=100 velocity=100, mimic joint=R_Middle_Flexor multiplier=1 offset=0
- added joint R_Middle_Flexor: type revolute, parent Middle_Knuckle_1, child Middle_Middle_1, origin xyz=-0.004 0.00265 0.045 rpy=0 0 0, axis -0.0 1.0 -0.0, limit lower=0.0 upper=1.047198 effort=100 velocity=100
- added joint R_Middle_Pitch: type revolute, parent Middle_Knuckle_Cross_1, child Middle_Knuckle_1, origin xyz=-0.0075 0.0048 0.004 rpy=0 0 0, axis -0.0 1.0 -0.0, limit lower=0.0 upper=1.308997 effort=100 velocity=100
- added joint R_Middle_Yaw: type revolute, parent Palm_1, child Middle_Knuckle_Cross_1, origin xyz=0.017 0.02875 0.090983 rpy=0 0 0, axis 1.0 0.0 0.0, limit lower=-0.349066 upper=0.349066 effort=100 velocity=100
- added joint R_Pinky_DIP: type revolute, parent Pinky_Middle_1, child Pinky_Tip_1, origin xyz=0.001397 -0.004132 0.029977 rpy=0 0 0, axis -0.178318 0.983965 0.003854, limit lower=0.0 upper=1.047198 effort=100 velocity=100, mimic joint=R_Pinky_Flexor multiplier=1 offset=0
- added joint R_Pinky_Flexor: type revolute, parent Pinky_Knuckle_1, child Pinky_Middle_1, origin xyz=-0.003435 0.001894 0.045085 rpy=0 0 0, axis -0.178318 0.983965 0.003854, limit lower=0.0 upper=1.047198 effort=100 velocity=100
- added joint R_Pinky_Pitch: type revolute, parent Pinky_Knuckle_Cross_1, child Pinky_Knuckle_1, origin xyz=-0.008147 0.003385 0.004177 rpy=0 0 0, axis -0.178318 0.983965 0.003854, limit lower=0.0 upper=1.308997 effort=100 velocity=100
- added joint R_Pinky_Yaw: type revolute, parent Palm_1, child Pinky_Knuckle_Cross_1, origin xyz=0.021743 -0.014307 0.078606 rpy=0 0 0, axis 0.983736 0.178359 -0.021263, limit lower=-0.349066 upper=0.349066 effort=100 velocity=100
- added joint R_Rigid 28: type fixed, parent Cobot_Forearm_1, child Solid_Wrist_1, origin xyz=0.0322 0.008656 -0.009117 rpy=0 0 0
- added joint R_Rigid 30: type fixed, parent Solid_Wrist_1, child Palm_1, origin xyz=-0.036054 -0.030102 0.143112 rpy=0 0 0
- added joint R_Rigid 31: type fixed, parent base_link, child Cobot_Forearm_1, origin xyz=0.0 0.0 0.008 rpy=0 0 0
- added joint R_Ring_DIP: type revolute, parent Ring_Middle_1, child Ring_Tip_1, origin xyz=0.000259 -0.004184 0.030001 rpy=0 0 0, axis -0.08702 0.996207 -0.00031, limit lower=0.0 upper=1.047198 effort=100 velocity=100, mimic joint=R_Ring_Flexor multiplier=1 offset=0
- added joint R_Ring_Flexor: type revolute, parent Ring_Knuckle_1, child Ring_Middle_1, origin xyz=-0.004376 0.002292 0.044985 rpy=0 0 0, axis -0.08702 0.996207 -0.00031, limit lower=0.0 upper=1.047198 effort=100 velocity=100
- added joint R_Ring_Pitch: type revolute, parent Ring_Knuckle_Cross_1, child Ring_Knuckle_1, origin xyz=-0.007904 0.004129 0.003971 rpy=0 0 0, axis -0.08702 0.996207 -0.00031, limit lower=0.0 upper=1.308997 effort=100 velocity=100
- added joint R_Ring_Yaw: type revolute, parent Palm_1, child Ring_Knuckle_Cross_1, origin xyz=0.018517 0.006437 0.08714 rpy=0 0 0, axis 0.9962 0.08702 0.003551, limit lower=-0.349066 upper=0.349066 effort=100 velocity=100
- added joint R_Thumb_DIP: type revolute, parent Thumb_Middle_1, child Thumb_Tip_1, origin xyz=0.031506 -0.000124 0.024645 rpy=0 0 0, axis 0.34773 -0.826541 -0.442622, limit lower=0.0 upper=1.047198 effort=100 velocity=100, mimic joint=R_Thumb_Flexor multiplier=1 offset=0
- added joint R_Thumb_Flexor: type revolute, parent Thumb_Knuckle_1, child Thumb_Middle_1, origin xyz=0.046855 -0.010807 0.021295 rpy=0 0 0, axis 0.34773 -0.826541 -0.442622, limit lower=0.0 upper=1.047198 effort=100 velocity=100
- added joint R_Thumb_Pitch: type revolute, parent Thumb_Dist_KC_1, child Thumb_Knuckle_1, origin xyz=0.005242 0.0081 0.011133 rpy=0 0 0, axis 0.34773 -0.826541 -0.442622, limit lower=0.0 upper=1.047198 effort=100 velocity=100
- added joint R_Thumb_Roll: type revolute, parent Thumb_Prox_KC_1, child Thumb_Dist_KC_1, origin xyz=-0.007225 -0.005798 0.00515 rpy=0 0 0, axis 0.786356 0.0 0.617773, limit lower=-0.349066 upper=0.349066 effort=100 velocity=100
- added joint R_Thumb_Yaw: type revolute, parent Palm_1, child Thumb_Prox_KC_1, origin xyz=0.042207 0.039244 -0.001357 rpy=0 0 0, axis 0.510615 0.562877 -0.649955, limit lower=-0.523599 upper=0.523599 effort=100 velocity=100

File: urdf/dexhandv2_cobot_right.xacro (robot description, xacro)
@@ -504,5 +504,5 @@
   </collision>
 </link>
-<joint name="Index_Pitch" type="revolute">
+<joint name="R_Index_Pitch" type="revolute">
   <origin xyz="-0.007032 0.005438 0.004034" rpy="0 0 0"/>
   <parent link="Index_Knuckle_Cross_1"/>
@@ -511,5 +511,5 @@
   <limit upper="1.308997" lower="0.0" effort="100" velocity="100"/>
 </joint>
-<joint name="Middle_Pitch" type="revolute">
+<joint name="R_Middle_Pitch" type="revolute">
   <origin xyz="-0.0075 0.0048 0.004" rpy="0 0 0"/>
   <parent link="Middle_Knuckle_Cross_1"/>
@@ -518,5 +518,5 @@
   <limit upper="1.308997" lower="0.0" effort="100" velocity="100"/>
 </joint>
-<joint name="Ring_Pitch" type="revolute">
+<joint name="R_Ring_Pitch" type="revolute">
   <origin xyz="-0.007904 0.004129 0.003971" rpy="0 0 0"/>
   <parent link="Ring_Knuckle_Cross_1"/>
@@ -525,5 +525,5 @@
   <limit upper="1.308997" lower="0.0" effort="100" velocity="100"/>
 </joint>
-<joint name="Pinky_Pitch" type="revolute">
+<joint name="R_Pinky_Pitch" type="revolute">
   <origin xyz="-0.008147 0.003385 0.004177" rpy="0 0 0"/>
   <parent link="Pinky_Knuckle_Cross_1"/>
@@ -532,5 +532,5 @@
   <limit upper="1.308997" lower="0.0" effort="100" velocity="100"/>
 </joint>
-<joint name="Index_PIP" type="revolute">
+<joint name="R_Index_Flexor" type="revolute">
   <origin xyz="-0.003532 0.002993 0.045018" rpy="0 0 0"/>
   <parent link="Index_Knuckle_1"/>
@@ -538,6 +538,6 @@
   <axis xyz="0.087537 0.996161 -0.000428"/>
   <limit upper="1.047198" lower="0.0" effort="100" velocity="100"/>
-</joint>
-<joint name="Middle_PIP" type="revolute">
+  </joint>
+<joint name="R_Middle_Flexor" type="revolute">
   <origin xyz="-0.004 0.00265 0.045" rpy="0 0 0"/>
   <parent link="Middle_Knuckle_1"/>
@@ -546,5 +546,5 @@
   <limit upper="1.047198" lower="0.0" effort="100" velocity="100"/>
 </joint>
-<joint name="Ring_PIP" type="revolute">
+<joint name="R_Ring_Flexor" type="revolute">
   <origin xyz="-0.004376 0.002292 0.044985" rpy="0 0 0"/>
   <parent link="Ring_Knuckle_1"/>
@@ -553,5 +553,5 @@
   <limit upper="1.047198" lower="0.0" effort="100" velocity="100"/>
 </joint>
-<joint name="Pinky_PIP" type="revolute">
+<joint name="R_Pinky_Flexor" type="revolute">
   <origin xyz="-0.003435 0.001894 0.045085" rpy="0 0 0"/>
   <parent link="Pinky_Knuckle_1"/>
@@ -560,5 +560,5 @@
   <limit upper="1.047198" lower="0.0" effort="100" velocity="100"/>
 </joint>
-<joint name="Index_DIP" type="revolute">
+<joint name="R_Index_DIP" type="revolute">
   <origin xyz="-0.000221 -0.004184 0.030002" rpy="0 0 0"/>
   <parent link="Index_Middle_1"/>
@@ -566,6 +566,7 @@
   <axis xyz="0.087537 0.996161 -0.000428"/>
   <limit upper="1.047198" lower="0.0" effort="100" velocity="100"/>
-</joint>
-<joint name="Middle_DIP" type="revolute">
+  <mimic joint="R_Index_Flexor" multiplier="1" offset="0"/>
+</joint>
+<joint name="R_Middle_DIP" type="revolute">
   <origin xyz="0.0 -0.0042 0.03" rpy="0 0 0"/>
   <parent link="Middle_Middle_1"/>
@@ -573,6 +574,7 @@
   <axis xyz="-0.0 1.0 -0.0"/>
   <limit upper="1.047198" lower="0.0" effort="100" velocity="100"/>
-</joint>
-<joint name="Ring_DIP" type="revolute">
+  <mimic joint="R_Middle_Flexor" multiplier="1" offset="0"/>
+</joint>
+<joint name="R_Ring_DIP" type="revolute">
   <origin xyz="0.000259 -0.004184 0.030001" rpy="0 0 0"/>
   <parent link="Ring_Middle_1"/>
@@ -580,6 +582,7 @@
   <axis xyz="-0.08702 0.996207 -0.00031"/>
   <limit upper="1.047198" lower="0.0" effort="100" velocity="100"/>
-</joint>
-<joint name="Pinky_DIP" type="revolute">
+  <mimic joint="R_Ring_Flexor" multiplier="1" offset="0"/>
+</joint>
+<joint name="R_Pinky_DIP" type="revolute">
   <origin xyz="0.001397 -0.004132 0.029977" rpy="0 0 0"/>
   <parent link="Pinky_Middle_1"/>
@@ -587,6 +590,7 @@
   <axis xyz="-0.178318 0.983965 0.003854"/>
   <limit upper="1.047198" lower="0.0" effort="100" velocity="100"/>
-</joint>
-<joint name="Thumb_Yaw" type="revolute">
+  <mimic joint="R_Pinky_Flexor" multiplier="1" offset="0"/>
+</joint>
+<joint name="R_Thumb_Yaw" type="revolute">
   <origin xyz="0.042207 0.039244 -0.001357" rpy="0 0 0"/>
   <parent link="Palm_1"/>
@@ -595,5 +599,5 @@
   <limit upper="0.523599" lower="-0.523599" effort="100" velocity="100"/>
 </joint>
-<joint name="Thumb_Roll" type="revolute">
+<joint name="R_Thumb_Roll" type="revolute">
   <origin xyz="-0.007225 -0.005798 0.00515" rpy="0 0 0"/>
   <parent link="Thumb_Prox_KC_1"/>
@@ -602,5 +606,5 @@
   <limit upper="0.349066" lower="-0.349066" effort="100" velocity="100"/>
 </joint>
-<joint name="Thumb_PIP" type="revolute">
+<joint name="R_Thumb_Flexor" type="revolute">
   <origin xyz="0.046855 -0.010807 0.021295" rpy="0 0 0"/>
   <parent link="Thumb_Knuckle_1"/>
@@ -609,5 +613,5 @@
   <limit upper="1.047198" lower="0.0" effort="100" velocity="100"/>
 </joint>
-<joint name="Thumb_DIP" type="revolute">
+<joint name="R_Thumb_DIP" type="revolute">
   <origin xyz="0.031506 -0.000124 0.024645" rpy="0 0 0"/>
   <parent link="Thumb_Middle_1"/>
@@ -615,6 +619,7 @@
   <axis xyz="0.34773 -0.826541 -0.442622"/>
   <limit upper="1.047198" lower="0.0" effort="100" velocity="100"/>
-</joint>
-<joint name="Index_Yaw" type="revolute">
+  <mimic joint="R_Thumb_Flexor" multiplier="1" offset="0"/>
+</joint>
+<joint name="R_Index_Yaw" type="revolute">
   <origin xyz="0.01778 0.050623 0.084894" rpy="0 0 0"/>
   <parent link="Palm_1"/>
@@ -623,5 +628,5 @@
   <limit upper="0.349066" lower="-0.349066" effort="100" velocity="100"/>
 </joint>
-<joint name="Middle_Yaw" type="revolute">
+<joint name="R_Middle_Yaw" type="revolute">
   <origin xyz="0.017 0.02875 0.090983" rpy="0 0 0"/>
   <parent link="Palm_1"/>
@@ -630,5 +635,5 @@
   <limit upper="0.349066" lower="-0.349066" effort="100" velocity="100"/>
 </joint>
-<joint name="Ring_Yaw" type="revolute">
+<joint name="R_Ring_Yaw" type="revolute">
   <origin xyz="0.018517 0.006437 0.08714" rpy="0 0 0"/>
   <parent link="Palm_1"/>
@@ -637,5 +642,5 @@
   <limit upper="0.349066" lower="-0.349066" effort="100" velocity="100"/>
 </joint>
-<joint name="Pinky_Yaw" type="revolute">
+<joint name="R_Pinky_Yaw" type="revolute">
   <origin xyz="0.021743 -0.014307 0.078606" rpy="0 0 0"/>
   <parent link="Palm_1"/>
@@ -644,5 +649,5 @@
   <limit upper="0.349066" lower="-0.349066" effort="100" velocity="100"/>
 </joint>
-<joint name="Thumb_Pitch" type="revolute">
+<joint name="R_Thumb_Pitch" type="revolute">
   <origin xyz="0.005242 0.0081 0.011133" rpy="0 0 0"/>
   <parent link="Thumb_Dist_KC_1"/>
@@ -651,15 +656,15 @@
   <limit upper="1.047198" lower="0.0" effort="100" velocity="100"/>
 </joint>
-<joint name="Rigid 28" type="fixed">
+<joint name="R_Rigid 28" type="fixed">
   <origin xyz="0.0322 0.008656 -0.009117" rpy="0 0 0"/>
   <parent link="Cobot_Forearm_1"/>
   <child link="Solid_Wrist_1"/>
 </joint>
-<joint name="Rigid 30" type="fixed">
+<joint name="R_Rigid 30" type="fixed">
   <origin xyz="-0.036054 -0.030102 0.143112" rpy="0 0 0"/>
   <parent link="Solid_Wrist_1"/>
   <child link="Palm_1"/>
 </joint>
-<joint name="Rigid 31" type="fixed">
+<joint name="R_Rigid 31" type="fixed">
   <origin xyz="0.0 0.0 0.008" rpy="0 0 0"/>
   <parent link="base_link"/>

File: urdf/dexhandv2_right.urdf (robot description, URDF)
Before this commit: robot dexhandv2_right, 22 links, 21 joints
Joints:
- removed joint Index_DIP
- removed joint Index_PIP
- removed joint Index_Pitch
- removed joint Index_Yaw
- removed joint Middle_DIP
- removed joint Middle_PIP
- removed joint Middle_Pitch
- removed joint Middle_Yaw
- removed joint Pinky_DIP
- removed joint Pinky_PIP
- removed joint Pinky_Pitch
- removed joint Pinky_Yaw
- removed joint Ring_DIP
- removed joint Ring_PIP
- removed joint Ring_Pitch
- removed joint Ring_Yaw
- removed joint Thumb_DIP
- removed joint Thumb_PIP
- removed joint Thumb_Pitch
- removed joint Thumb_Roll
- removed joint Thumb_Yaw
- added joint R_Index_DIP: type revolute, parent Index_Middle_1, child Index_Tip_1, origin xyz=-0.000221 -0.004184 0.030001 rpy=0 0 0, axis 0.087537 0.996161 -0.000428, limit lower=0.0 upper=1.047198 effort=100 velocity=100, mimic joint=Index_Flexor multiplier=1 offset=0
- added joint R_Index_Flexor: type revolute, parent Index_Knuckle_1, child Index_Middle_1, origin xyz=-0.003532 0.002993 0.045018 rpy=0 0 0, axis 0.087537 0.996161 -0.000428, limit lower=0.0 upper=1.047198 effort=100 velocity=100
- added joint R_Index_Pitch: type revolute, parent Index_Knuckle_Cross_1, child Index_Knuckle_1, origin xyz=-0.007032 0.005438 0.004034 rpy=0 0 0, axis 0.087537 0.996161 -0.000428, limit lower=0.0 upper=1.308997 effort=100 velocity=100
- added joint R_Index_Yaw: type revolute, parent base_link, child Index_Knuckle_Cross_1, origin xyz=0.01778 0.029123 0.084894 rpy=0 0 0, axis 0.996149 -0.087538 -0.004875, limit lower=-0.349066 upper=0.349066 effort=100 velocity=100
- added joint R_Middle_DIP: type revolute, parent Middle_Middle_1, child Midle_Tip_1, origin xyz=0.0 -0.0042 0.03 rpy=0 0 0, axis -0.0 1.0 0.0, limit lower=0.0 upper=1.047198 effort=100 velocity=100, mimic joint=Middle_Flexor multiplier=1 offset=0
- added joint R_Middle_Flexor: type revolute, parent Middle_Knuckle_1, child Middle_Middle_1, origin xyz=-0.004 0.00265 0.045 rpy=0 0 0, axis -0.0 1.0 0.0, limit lower=0.0 upper=1.047198 effort=100 velocity=100
- added joint R_Middle_Pitch: type revolute, parent Middle_Knuckle_Cross_1, child Middle_Knuckle_1, origin xyz=-0.0075 0.0048 0.004 rpy=0 0 0, axis -0.0 1.0 0.0, limit lower=0.0 upper=1.308997 effort=100 velocity=100
- added joint R_Middle_Yaw: type revolute, parent base_link, child Middle_Knuckle_Cross_1, origin xyz=0.017 0.00725 0.090983 rpy=0 0 0, axis 1.0 0.0 -0.0, limit lower=-0.349066 upper=0.349066 effort=100 velocity=100
- added joint R_Pinky_DIP: type revolute, parent Pinky_Middle_1, child Pinky_Tip_1, origin xyz=0.001397 -0.004132 0.029977 rpy=0 0 0, axis -0.178318 0.983965 0.003854, limit lower=0.0 upper=1.047198 effort=100 velocity=100, mimic joint=Pinky_Flexor multiplier=1 offset=0
- added joint R_Pinky_Flexor: type revolute, parent Pinky_Knuckle_1, child Pinky_Middle_1, origin xyz=-0.003435 0.001894 0.045085 rpy=0 0 0, axis -0.178318 0.983965 0.003854, limit lower=0.0 upper=1.047198 effort=100 velocity=100
- added joint R_Pinky_Pitch: type revolute, parent Pinky_Knuckle_Cross_1, child Pinky_Knuckle_1, origin xyz=-0.008147 0.003385 0.004177 rpy=0 0 0, axis -0.178318 0.983965 0.003854, limit lower=0.0 upper=1.308997 effort=100 velocity=100
- added joint R_Pinky_Yaw: type revolute, parent base_link, child Pinky_Knuckle_Cross_1, origin xyz=0.021743 -0.035807 0.078606 rpy=0 0 0, axis 0.983736 0.178359 -0.021263, limit lower=-0.349066 upper=0.349066 effort=100 velocity=100
- added joint R_Ring_DIP: type revolute, parent Ring_Middle_1, child Ring_Tip_1, origin xyz=0.000259 -0.004184 0.030001 rpy=0 0 0, axis -0.08702 0.996207 -0.00031, limit lower=0.0 upper=1.047198 effort=100 velocity=100, mimic joint=Ring_Flexor multiplier=1 offset=0
- added joint R_Ring_Flexor: type revolute, parent Ring_Knuckle_1, child Ring_Middle_1, origin xyz=-0.004376 0.002292 0.044985 rpy=0 0 0, axis -0.08702 0.996207 -0.00031, limit lower=0.0 upper=1.047198 effort=100 velocity=100
- added joint R_Ring_Pitch: type revolute, parent Ring_Knuckle_Cross_1, child Ring_Knuckle_1, origin xyz=-0.007904 0.004129 0.003972 rpy=0 0 0, axis -0.08702 0.996207 -0.00031, limit lower=0.0 upper=1.308997 effort=100 velocity=100
- added joint R_Ring_Yaw: type revolute, parent base_link, child Ring_Knuckle_Cross_1, origin xyz=0.018517 -0.015063 0.087139 rpy=0 0 0, axis 0.9962 0.08702 0.003551, limit lower=-0.349066 upper=0.349066 effort=100 velocity=100
- added joint R_Thumb_DIP: type revolute, parent Thumb_Middle_1, child Thumb_Tip_1, origin xyz=0.031506 -0.000124 0.024645 rpy=0 0 0, axis 0.34773 -0.826541 -0.442622, limit lower=0.0 upper=1.047198 effort=100 velocity=100, mimic joint=Thumb_Flexor multiplier=1 offset=0
- added joint R_Thumb_Flexor: type revolute, parent Thumb_Knuckle_1, child Thumb_Middle_1, origin xyz=0.046855 -0.010808 0.021295 rpy=0 0 0, axis 0.34773 -0.826541 -0.442622, limit lower=0.0 upper=1.047198 effort=100 velocity=100
- added joint R_Thumb_Pitch: type revolute, parent Thumb_Dist_KC_1, child Thumb_Knuckle_1, origin xyz=0.005242 0.0081 0.011134 rpy=0 0 0, axis 0.34773 -0.826541 -0.442622, limit lower=0.0 upper=1.047198 effort=100 velocity=100
- added joint R_Thumb_Roll: type revolute, parent Thumb_Prox_KC_1, child Thumb_Dist_KC_1, origin xyz=-0.007225 -0.005798 0.00515 rpy=0 0 0, axis 0.786356 -0.0 0.617773, limit lower=-0.349066 upper=0.349066 effort=100 velocity=100
- added joint R_Thumb_Yaw: type revolute, parent base_link, child Thumb_Prox_KC_1, origin xyz=0.042207 0.017744 -0.001358 rpy=0 0 0, axis 0.510615 0.562877 -0.649955, limit lower=-0.523599 upper=0.523599 effort=100 velocity=100
