Commit message: V0.0.2 - Created mimic constraint between first two joints of each finger, and renamed the joints to _Flexor to reflect actual mechanics.

File: urdf/dexhandv2_right.xacro (robot description, xacro)
@@ -444,5 +444,5 @@
   </collision>
 </link>
-<joint name="Index_Pitch" type="revolute">
+<joint name="R_Index_Pitch" type="revolute">
   <origin xyz="-0.007032 0.005438 0.004034" rpy="0 0 0"/>
   <parent link="Index_Knuckle_Cross_1"/>
@@ -451,5 +451,5 @@
   <limit upper="1.308997" lower="0.0" effort="100" velocity="100"/>
 </joint>
-<joint name="Middle_Pitch" type="revolute">
+<joint name="R_Middle_Pitch" type="revolute">
   <origin xyz="-0.0075 0.0048 0.004" rpy="0 0 0"/>
   <parent link="Middle_Knuckle_Cross_1"/>
@@ -458,5 +458,5 @@
   <limit upper="1.308997" lower="0.0" effort="100" velocity="100"/>
 </joint>
-<joint name="Ring_Pitch" type="revolute">
+<joint name="R_Ring_Pitch" type="revolute">
   <origin xyz="-0.007904 0.004129 0.003972" rpy="0 0 0"/>
   <parent link="Ring_Knuckle_Cross_1"/>
@@ -465,5 +465,5 @@
   <limit upper="1.308997" lower="0.0" effort="100" velocity="100"/>
 </joint>
-<joint name="Pinky_Pitch" type="revolute">
+<joint name="R_Pinky_Pitch" type="revolute">
   <origin xyz="-0.008147 0.003385 0.004177" rpy="0 0 0"/>
   <parent link="Pinky_Knuckle_Cross_1"/>
@@ -472,5 +472,5 @@
   <limit upper="1.308997" lower="0.0" effort="100" velocity="100"/>
 </joint>
-<joint name="Index_PIP" type="revolute">
+<joint name="R_Index_Flexor" type="revolute">
   <origin xyz="-0.003532 0.002993 0.045018" rpy="0 0 0"/>
   <parent link="Index_Knuckle_1"/>
@@ -479,5 +479,5 @@
   <limit upper="1.047198" lower="0.0" effort="100" velocity="100"/>
 </joint>
-<joint name="Middle_PIP" type="revolute">
+<joint name="R_Middle_Flexor" type="revolute">
   <origin xyz="-0.004 0.00265 0.045" rpy="0 0 0"/>
   <parent link="Middle_Knuckle_1"/>
@@ -486,5 +486,5 @@
   <limit upper="1.047198" lower="0.0" effort="100" velocity="100"/>
 </joint>
-<joint name="Ring_PIP" type="revolute">
+<joint name="R_Ring_Flexor" type="revolute">
   <origin xyz="-0.004376 0.002292 0.044985" rpy="0 0 0"/>
   <parent link="Ring_Knuckle_1"/>
@@ -493,5 +493,5 @@
   <limit upper="1.047198" lower="0.0" effort="100" velocity="100"/>
 </joint>
-<joint name="Pinky_PIP" type="revolute">
+<joint name="R_Pinky_Flexor" type="revolute">
   <origin xyz="-0.003435 0.001894 0.045085" rpy="0 0 0"/>
   <parent link="Pinky_Knuckle_1"/>
@@ -500,5 +500,5 @@
   <limit upper="1.047198" lower="0.0" effort="100" velocity="100"/>
 </joint>
-<joint name="Index_DIP" type="revolute">
+<joint name="R_Index_DIP" type="revolute">
   <origin xyz="-0.000221 -0.004184 0.030001" rpy="0 0 0"/>
   <parent link="Index_Middle_1"/>
@@ -506,6 +506,7 @@
   <axis xyz="0.087537 0.996161 -0.000428"/>
   <limit upper="1.047198" lower="0.0" effort="100" velocity="100"/>
-</joint>
-<joint name="Middle_DIP" type="revolute">
+  <mimic joint="Index_Flexor" multiplier="1" offset="0"/>
+</joint>
+<joint name="R_Middle_DIP" type="revolute">
   <origin xyz="0.0 -0.0042 0.03" rpy="0 0 0"/>
   <parent link="Middle_Middle_1"/>
@@ -513,6 +514,7 @@
   <axis xyz="-0.0 1.0 0.0"/>
   <limit upper="1.047198" lower="0.0" effort="100" velocity="100"/>
-</joint>
-<joint name="Ring_DIP" type="revolute">
+  <mimic joint="Middle_Flexor" multiplier="1" offset="0"/>
+</joint>
+<joint name="R_Ring_DIP" type="revolute">
   <origin xyz="0.000259 -0.004184 0.030001" rpy="0 0 0"/>
   <parent link="Ring_Middle_1"/>
@@ -520,6 +522,7 @@
   <axis xyz="-0.08702 0.996207 -0.00031"/>
   <limit upper="1.047198" lower="0.0" effort="100" velocity="100"/>
-</joint>
-<joint name="Pinky_DIP" type="revolute">
+  <mimic joint="Ring_Flexor" multiplier="1" offset="0"/>
+</joint>
+<joint name="R_Pinky_DIP" type="revolute">
   <origin xyz="0.001397 -0.004132 0.029977" rpy="0 0 0"/>
   <parent link="Pinky_Middle_1"/>
@@ -527,6 +530,7 @@
   <axis xyz="-0.178318 0.983965 0.003854"/>
   <limit upper="1.047198" lower="0.0" effort="100" velocity="100"/>
-</joint>
-<joint name="Thumb_Yaw" type="revolute">
+  <mimic joint="Pinky_Flexor" multiplier="1" offset="0"/>
+</joint>
+<joint name="R_Thumb_Yaw" type="revolute">
   <origin xyz="0.042207 0.017744 -0.001358" rpy="0 0 0"/>
   <parent link="base_link"/>
@@ -535,5 +539,5 @@
   <limit upper="0.523599" lower="-0.523599" effort="100" velocity="100"/>
 </joint>
-<joint name="Thumb_Roll" type="revolute">
+<joint name="R_Thumb_Roll" type="revolute">
   <origin xyz="-0.007225 -0.005798 0.00515" rpy="0 0 0"/>
   <parent link="Thumb_Prox_KC_1"/>
@@ -542,5 +546,5 @@
   <limit upper="0.349066" lower="-0.349066" effort="100" velocity="100"/>
 </joint>
-<joint name="Thumb_PIP" type="revolute">
+<joint name="R_Thumb_Flexor" type="revolute">
   <origin xyz="0.046855 -0.010808 0.021295" rpy="0 0 0"/>
   <parent link="Thumb_Knuckle_1"/>
@@ -549,5 +553,5 @@
   <limit upper="1.047198" lower="0.0" effort="100" velocity="100"/>
 </joint>
-<joint name="Thumb_DIP" type="revolute">
+<joint name="R_Thumb_DIP" type="revolute">
   <origin xyz="0.031506 -0.000124 0.024645" rpy="0 0 0"/>
   <parent link="Thumb_Middle_1"/>
@@ -555,6 +559,7 @@
   <axis xyz="0.34773 -0.826541 -0.442622"/>
   <limit upper="1.047198" lower="0.0" effort="100" velocity="100"/>
-</joint>
-<joint name="Index_Yaw" type="revolute">
+  <mimic joint="Thumb_Flexor" multiplier="1" offset="0"/>
+</joint>
+<joint name="R_Index_Yaw" type="revolute">
   <origin xyz="0.01778 0.029123 0.084894" rpy="0 0 0"/>
   <parent link="base_link"/>
@@ -563,5 +568,5 @@
   <limit upper="0.349066" lower="-0.349066" effort="100" velocity="100"/>
 </joint>
-<joint name="Middle_Yaw" type="revolute">
+<joint name="R_Middle_Yaw" type="revolute">
   <origin xyz="0.017 0.00725 0.090983" rpy="0 0 0"/>
   <parent link="base_link"/>
@@ -570,5 +575,5 @@
   <limit upper="0.349066" lower="-0.349066" effort="100" velocity="100"/>
 </joint>
-<joint name="Ring_Yaw" type="revolute">
+<joint name="R_Ring_Yaw" type="revolute">
   <origin xyz="0.018517 -0.015063 0.087139" rpy="0 0 0"/>
   <parent link="base_link"/>
@@ -577,5 +582,5 @@
   <limit upper="0.349066" lower="-0.349066" effort="100" velocity="100"/>
 </joint>
-<joint name="Pinky_Yaw" type="revolute">
+<joint name="R_Pinky_Yaw" type="revolute">
   <origin xyz="0.021743 -0.035807 0.078606" rpy="0 0 0"/>
   <parent link="base_link"/>
@@ -584,5 +589,5 @@
   <limit upper="0.349066" lower="-0.349066" effort="100" velocity="100"/>
 </joint>
-<joint name="Thumb_Pitch" type="revolute">
+<joint name="R_Thumb_Pitch" type="revolute">
   <origin xyz="0.005242 0.0081 0.011134" rpy="0 0 0"/>
   <parent link="Thumb_Dist_KC_1"/>

Commit message: Updated range of motion on thumb yaw

File: urdf/dexhandv2_cobot_right.urdf (robot description, URDF)
Before this commit: robot dexhandv2_cobot_right, 25 links, 24 joints
Joints:
- joint R_Thumb_Yaw: limit lower=-0.523599 upper=0.523599 effort=100 velocity=100 -> lower=-0.523599 upper=0.0872665 effort=100 velocity=100

File: urdf/dexhandv2_cobot_right.xacro (robot description, xacro)
@@ -597,5 +597,5 @@
   <child link="Thumb_Prox_KC_1"/>
   <axis xyz="0.510615 0.562877 -0.649955"/>
-  <limit upper="0.523599" lower="-0.523599" effort="100" velocity="100"/>
+  <limit upper="0.0872665" lower="-0.523599" effort="100" velocity="100"/>
 </joint>
 <joint name="R_Thumb_Roll" type="revolute">
